File: uvLed/_autosave-uvLed.kicad_sch (KiCad schematic)
At the start: 10 parts, among them J1 Conn_01x02

Commit message: update pcb
Connections:
- net GND: now also D8.1 (K); no longer D5.1 (K)
- net at D7.1 (K): now also D8.2 (A); no longer D6.2 (A)
- net at D7.2 (A): now also D6.1 (K); no longer D8.1 (K)
- net at C1.1, D4.2 (A), J1.1 (Pin_1): now also D5.2 (A); no longer D8.2 (A)
- new net: D5.1 (K), D6.2 (A)
Other:
- moved on the sheet: D5, D6, D7, D8
Changed lines of the file:
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@@
 (kicad_sch (version 20230121) (generator eeschema)
   (paper "A4")
-  (junction (at 167.64 91.44) (diameter 0) (color 0 0 0 0)
-  )
   (junction (at 171.45 83.82) (diameter 0) (color 0 0 0 0)
   )
-  (junction (at 163.83 88.9) (diameter 0) (color 0 0 0 0)
+  (junction (at 163.83 91.44) (diameter 0) (color 0 0 0 0)
   )
   (junction (at 171.45 91.44) (diameter 0) (color 0 0 0 0)
   )
-  (wire (pts (xy 167.64 104.14) (xy 167.64 91.44))
+  (junction (at 167.64 83.82) (diameter 0) (color 0 0 0 0)
+  )
+  (wire (pts (xy 167.64 83.82) (xy 167.64 104.14))
     (stroke (width 0) (type default))
   )
@@
     (stroke (width 0) (type default))
   )
+  (wire (pts (xy 120.65 104.14) (xy 167.64 104.14))
+    (stroke (width 0) (type default))
+  )
   (wire (pts (xy 129.54 100.33) (xy 133.35 100.33))
     (stroke (width 0) (type default))
   )
-  (wire (pts (xy 171.45 83.82) (xy 163.83 83.82))
+  (wire (pts (xy 171.45 83.82) (xy 167.64 83.82))
     (stroke (width 0) (type default))
   )
@@
     (stroke (width 0) (type default))
   )
+  (wire (pts (xy 167.64 83.82) (xy 163.83 83.82))
+    (stroke (width 0) (type default))
+  )
   (wire (pts (xy 177.8 88.9) (xy 177.8 83.82))
     (stroke (width 0) (type default))
@@
     (stroke (width 0) (type default))
   )
-  (wire (pts (xy 163.83 88.9) (xy 163.83 100.33))
-    (stroke (width 0) (type default))
-  )
   (wire (pts (xy 120.65 100.33) (xy 120.65 104.14))
     (stroke (width 0) (type default))
@@
     (stroke (width 0) (type default))
   )
-  (wire (pts (xy 167.64 91.44) (xy 171.45 91.44))
-    (stroke (width 0) (type default))
-  )
-  (wire (pts (xy 120.65 104.14) (xy 167.64 104.14))
-    (stroke (width 0) (type default))
-  )
-  (wire (pts (xy 120.65 91.44) (xy 167.64 91.44))
+  (wire (pts (xy 120.65 91.44) (xy 163.83 91.44))
+    (stroke (width 0) (type default))
+  )
+  (wire (pts (xy 163.83 91.44) (xy 171.45 91.44))
+    (stroke (width 0) (type default))
+  )
+  (wire (pts (xy 163.83 91.44) (xy 163.83 100.33))
     (stroke (width 0) (type default))
   )
@@
     )
   )
-  (symbol (lib_id "Device:LED") (at 148.59 100.33 0) (unit 1)
-    (in_bom yes) (on_board yes) (dnp no) (fields_autoplaced)
-    (property "Reference" "D7" (at 147.0025 93.98 0)
-      (effects (font (size 1.27 1.27)))
-    )
-    (property "Value" "LED" (at 147.0025 96.52 0)
+  (symbol (lib_id "Device:LED") (at 148.59 100.33 180) (unit 1)
+    (in_bom yes) (on_board yes) (dnp no) (fields_autoplaced)
+    (property "Reference" "D7" (at 150.1775 92.71 0)
+      (effects (font (size 1.27 1.27)))
+    )
+    (property "Value" "LED" (at 150.1775 95.25 0)
       (effects (font (size 1.27 1.27)))
     )
@@
     )
   )
-  (symbol (lib_id "Device:LED") (at 125.73 100.33 0) (unit 1)
-    (in_bom yes) (on_board yes) (dnp no) (fields_autoplaced)
-    (property "Reference" "D5" (at 124.1425 93.98 0)
-      (effects (font (size 1.27 1.27)))
-    )
-    (property "Value" "LED" (at 124.1425 96.52 0)
+  (symbol (lib_id "Device:LED") (at 125.73 100.33 180) (unit 1)
+    (in_bom yes) (on_board yes) (dnp no) (fields_autoplaced)
+    (property "Reference" "D5" (at 127.3175 92.71 0)
+      (effects (font (size 1.27 1.27)))
+    )
+    (property "Value" "LED" (at 127.3175 95.25 0)
       (effects (font (size 1.27 1.27)))
     )
@@
     )
   )
-  (symbol (lib_id "Device:LED") (at 160.02 100.33 0) (unit 1)
-    (in_bom yes) (on_board yes) (dnp no) (fields_autoplaced)
-    (property "Reference" "D8" (at 158.4325 93.98 0)
-      (effects (font (size 1.27 1.27)))
-    )
-    (property "Value" "LED" (at 158.4325 96.52 0)
+  (symbol (lib_id "Device:LED") (at 160.02 100.33 180) (unit 1)
+    (in_bom yes) (on_board yes) (dnp no) (fields_autoplaced)
+    (property "Reference" "D8" (at 161.6075 92.71 0)
+      (effects (font (size 1.27 1.27)))
+    )
+    (property "Value" "LED" (at 161.6075 95.25 0)
       (effects (font (size 1.27 1.27)))
     )
@@
     )
   )
-  (symbol (lib_id "Device:LED") (at 137.16 100.33 0) (unit 1)
-    (in_bom yes) (on_board yes) (dnp no) (fields_autoplaced)
-    (property "Reference" "D6" (at 135.5725 93.98 0)
-      (effects (font (size 1.27 1.27)))
-    )
-    (property "Value" "LED" (at 135.5725 96.52 0)
-      (effects (font (size 1.27 1.27)))
-    )
+  (symbol (lib_id "Device:LED") (at 137.16 100.33 180) (unit 1)
+    (in_bom yes) (on_board yes) (dnp no) (fields_autoplaced)
+    (property "Reference" "D6" (at 138.7475 92.71 0)
+      (effects (font (size 1.27 1.27)))
+    )
+    (property "Value" "LED" (at 138.7475 95.25 0)
+      (effects (font (size 1.27 1.27)))
+    )
